File: hw/servo/servo.kicad_sch (KiCad schematic)
At the start: 1 part, among them M1 Motor_Servo

Commit message: update schematics
Parts:
- renumbered M1 to M2
Connections:
- net +3.3V renamed +5V
- net D43 renamed D5
Changed lines of the file:
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@@
 	(generator_version "10.0")
 	(paper "A4")
-	(global_label "D43"
+	(global_label "D5"
 		(shape input)
 		(at 113.03 76.2 180)
@@
 		)
 		(property "Intersheetrefs" "${INTERSHEET_REFS}"
-			(at 106.3558 76.2 0)
+			(at 107.5653 76.2 0)
 			(hide yes)
 			(show_name no)
@@
 		(in_pos_files yes)
 		(dnp no)
-		(fields_autoplaced yes)
 		(property "Reference" "#PWR02"
 			(at 113.03 87.63 0)
@@
 		)
 		(property "Value" "GND"
-			(at 113.03 86.36 0)
+			(at 113.03 85.344 0)
 			(show_name no)
 			(do_not_autoplace no)
@@
 		(in_pos_files yes)
 		(dnp no)
-		(fields_autoplaced yes)
-		(property "Reference" "M1"
-			(at 129.54 77.0368 0)
+		(property "Reference" "M2"
+			(at 128.778 76.962 0)
 			(show_name no)
 			(do_not_autoplace no)
@@
 		)
 		(property "Value" "Motor_Servo"
-			(at 129.54 79.5768 0)
+			(at 128.778 79.502 0)
 			(show_name no)
 			(do_not_autoplace no)
@@
 			(project "servo"
 				(path "/afcc8374-9203-41d6-bdd1-3391cdab8afa"
-					(reference "M1")
+					(reference "M2")
 					(unit 1)
 				)
@@
 		(in_pos_files yes)
 		(dnp no)
-		(fields_autoplaced yes)
 		(property "Reference" "#PWR01"
 			(at 116.84 78.74 0)
@@
 			)
 		)
-		(property "Value" "+3.3V"
-			(at 109.22 78.7399 90)
-			(show_name no)
-			(do_not_autoplace no)
-			(effects
-				(font
-					(size 1.27 1.27)
-				)
-				(justify left)
-			)
-		)
+		(property "Value" "+5V"
+			(at 107.696 78.74 90)
+			(show_name no)
+			(do_not_autoplace no)
+			(effects
+				(font
+					(size 1.27 1.27)
+				)
+			)
+		)
