File: hw/valve/valve.kicad_sch (KiCad schematic)
At the start: 4 parts, among them J1 VALVE, Q1 IRLZ44N

Commit message: update schematics
Parts:
- Q1: value IRLZ44N -> IRLZ34N
Connections:
- net D33 renamed D6
Changed lines of the file:
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@@
 		)
 	)
-	(global_label "D33"
+	(global_label "D6"
 		(shape input)
 		(at 132.08 86.36 180)
@@
 		)
 		(property "Intersheetrefs" "${INTERSHEET_REFS}"
-			(at 125.4058 86.36 0)
+			(at 126.6153 86.36 0)
 			(hide yes)
 			(show_name no)
@@
 			)
 		)
-		(property "Value" "IRLZ44N"
+		(property "Value" "IRLZ34N"
 			(at 150.876 87.63 0)
 			(show_name no)
